Commit message: Changed .URDF file to attach the gripper on the arm

File: ur5_model/ur5_template.urdf (robot description, URDF)
Before this commit: robot ur5, 10 links, 9 joints
Links:
- added link simple_gripper_base; collision box size=0.03 0.04 0.06; collision cylinder length=0.045 radius=0.04
- added link simple_gripper_left_coupler; collision box size=0.03 0.065 0.02; visual mesh filename={}/gripper/meshes/visual/coupler.dae scale=0.001 0.001 0.001
- added link simple_gripper_left_driver; collision box size=0.02 0.04 0.02; visual mesh filename={}/gripper/meshes/visual/driver.dae scale=0.001 0.001 0.001
- added link simple_gripper_left_follower; collision box size=0.02 0.015 0.048; visual mesh filename={}/gripper/meshes/visual/follower.dae scale=0.001 0.001 0.001
- added link simple_gripper_left_pad; collision box size=0.02 0.008 0.036; visual mesh filename={}/gripper/meshes/visual/pad.dae scale=0.001 0.001 0.001
- added link simple_gripper_left_spring_link; collision box size=0.04 0.02 0.065; visual mesh filename={}/gripper/meshes/visual/spring_link.dae scale=0.001 0.001 0.001
- added link simple_gripper_right_coupler; collision box size=0.03 0.065 0.02; visual mesh filename={}/gripper/meshes/visual/coupler.dae scale=0.001 0.001 0.001
- added link simple_gripper_right_driver; collision box size=0.02 0.04 0.02; visual mesh filename={}/gripper/meshes/visual/driver.dae scale=0.001 0.001 0.001
- added link simple_gripper_right_follower; collision box size=0.02 0.015 0.048; visual mesh filename={}/gripper/meshes/visual/follower.dae scale=0.001 0.001 0.001
- added link simple_gripper_right_pad; collision box size=0.02 0.008 0.036; visual mesh filename={}/gripper/meshes/visual/pad.dae scale=0.001 0.001 0.001
- added link simple_gripper_right_spring_link; collision box size=0.04 0.02 0.065; visual mesh filename={}/gripper/meshes/visual/spring_link.dae scale=0.001 0.001 0.001
- link base_link: geometry collision mesh filename={}/arm/meshes/collision/base.stl; visual mesh filename={}/arm/meshes/visual/base.dae
- link forearm_link: geometry collision mesh filename={}/arm/meshes/collision/forearm.stl; visual mesh filename={}/arm/meshes/visual/forearm.dae
- link shoulder_link: geometry collision mesh filename={}/arm/meshes/collision/shoulder.stl; visual mesh filename={}/arm/meshes/visual/shoulder.dae
- link upper_arm_link: geometry collision mesh filename={}/arm/meshes/collision/upperarm.stl; visual mesh filename={}/arm/meshes/visual/upperarm.dae
- link wrist_1_link: geometry collision mesh filename={}/arm/meshes/collision/wrist1.stl; visual mesh filename={}/arm/meshes/visual/wrist1.dae
- link wrist_2_link: geometry collision mesh filename={}/arm/meshes/collision/wrist2.stl; visual mesh filename={}/arm/meshes/visual/wrist2.dae
- link wrist_3_link: geometry collision mesh filename={}/arm/meshes/collision/wrist3.stl; visual mesh filename={}/arm/meshes/visual/wrist3.dae
Joints:
- added joint Gripper_Adapter_Fix: type fixed, parent ee_link, child simple_gripper_base, origin xyz=0.0 0.0 0.0 rpy=0.0 1.57075 0.0
- added joint simple_gripper_left_coupler_joint: type fixed, parent simple_gripper_left_driver, child simple_gripper_left_coupler, origin xyz=0 0.0315 -0.0041 rpy=0 0 0
- added joint simple_gripper_left_driver_joint: type revolute, parent simple_gripper_base, child simple_gripper_left_driver, origin xyz=0 -0.0306011 0.054904 rpy=0 0 3.141592653589793, axis 1 0 0, limit lower=0.0 upper=0.715584844444 effort=176 velocity=1.91986177778, mimic joint=simple_gripper_right_driver_joint multiplier=1
- added joint simple_gripper_left_follower_joint: type revolute, parent simple_gripper_left_coupler, child simple_gripper_left_follower, origin xyz=0 0.0061 0.0471 rpy=0 0 0, axis 1 0 0, limit lower=-2.96705911111 upper=2.96705911111 effort=176 velocity=1.91986177778, mimic joint=simple_gripper_right_driver_joint multiplier=-1
- added joint simple_gripper_left_pad_joint: type fixed, parent simple_gripper_left_follower, child simple_gripper_left_pad
- added joint simple_gripper_left_spring_link_joint: type revolute, parent simple_gripper_base, child simple_gripper_left_spring_link, origin xyz=0 -0.012 0.0614 rpy=0 0 3.141592653589793, axis 1 0 0, limit lower=-2.96705911111 upper=2.96705911111 effort=176 velocity=1.91986177778, mimic joint=simple_gripper_right_driver_joint multiplier=1
- added joint simple_gripper_right_coupler_joint: type fixed, parent simple_gripper_right_driver, child simple_gripper_right_coupler, origin xyz=0 0.0315 -0.0041 rpy=0 0 0
- added joint simple_gripper_right_driver_joint: type revolute, parent simple_gripper_base, child simple_gripper_right_driver, origin xyz=0 0.0306011 0.054904 rpy=0 0 0, axis 1 0 0, limit lower=0.0 upper=0.872664444444 effort=60 velocity=1.91986177778
- added joint simple_gripper_right_follower_joint: type revolute, parent simple_gripper_right_coupler, child simple_gripper_right_follower, origin xyz=0 0.0061 0.0471 rpy=0 0 0, axis 1 0 0, limit lower=-2.96705911111 upper=2.96705911111 effort=176 velocity=1.91986177778, mimic joint=simple_gripper_right_driver_joint multiplier=-1
- added joint simple_gripper_right_pad_joint: type fixed, parent simple_gripper_right_follower, child simple_gripper_right_pad
- added joint simple_gripper_right_spring_link_joint: type revolute, parent simple_gripper_base, child simple_gripper_right_spring_link, origin xyz=0 0.012 0.0614 rpy=0 0 0, axis 1 0 0, limit lower=-2.96705911111 upper=2.96705911111 effort=176 velocity=1.91986177778, mimic joint=simple_gripper_right_driver_joint multiplier=1

Commit message: Corrected the positioning of tf for the end-effector

File: ur5_model/ur5_template.urdf (robot description, URDF)
Before this commit: robot ur5_robotiq_model, 21 links, 20 joints
Joints:
- joint Gripper_Adapter_Fix: origin xyz=0.0 0.0 0.0 rpy=0.0 1.57075 0.0 -> xyz=-0.08 0.0 0.0 rpy=0.0 1.57075 0.0
- joint ee_fixed_joint: origin xyz=0.0 0.0823 0.0 rpy=0.0 0.0 1.570796325 -> xyz=0.0 0.1623 0.0 rpy=0.0 0.0 1.570796325

Commit message: SRDF: Renamed the end-effector name to be consistent; URDF: Changed the name so SRDF and URDF match due to error popping up everytime the URDF/SRDF was loading.

File: ur5_model/ur5_template.urdf (robot description, URDF)
Before this commit: robot ur5_robotiq_model, 21 links, 20 joints
Joints:
- joint Gripper_Adapter_Fix: origin xyz=-0.08 0.0 0.0 rpy=0.0 1.57075 0.0 -> xyz=0.0 0.0 0.0 rpy=0.0 1.57075 0.0
- joint ee_fixed_joint: origin xyz=0.0 0.1623 0.0 rpy=0.0 0.0 1.570796325 -> xyz=0.0 0.0823 0.0 rpy=0.0 0.0 1.570796325
