Commit message: Refactored the URDF file to use package:// and renamed some folders

File: ur5_description/ur5.urdf (robot description, URDF)
Before this commit: robot ur5, 21 links, 20 joints
Links:
- link base_link: geometry collision mesh filename=package://ur5controller/ur5_description/arm/meshes/collisio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; visual mesh filename=package://ur5controller/ur5_description/arm/meshes/visual/b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
- link forearm_link: geometry collision mesh filename=package://ur5controller/ur5_description/arm/meshes/collisio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; visual mesh filename=package://ur5controller/ur5_description/arm/meshes/visual/f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
- link shoulder_link: geometry collision mesh filename=package://ur5controller/ur5_description/arm/meshes/collisio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; visual mesh filename=package://ur5controller/ur5_description/arm/meshes/visual/s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
- link simple_gripper_base: geometry collision box size=0.03 0.04 0.06; collision cylinder length=0.045 radius=0.04
- link simple_gripper_left_coupler: geometry collision box size=0.03 0.065 0.02; visual mesh filename=package://ur5controller/ur5_description/robotiq_two_finger_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 scale=0.001 0.001 0.001
- link simple_gripper_left_driver: geometry collision box size=0.02 0.04 0.02; visual mesh filename=package://ur5controller/ur5_description/robotiq_two_finger_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 scale=0.001 0.001 0.001
- link simple_gripper_left_follower: geometry collision box size=0.02 0.015 0.048; visual mesh filename=package://ur5controller/ur5_description/robotiq_two_finger_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 scale=0.001 0.001 0.001
- link simple_gripper_left_pad: geometry collision box size=0.02 0.008 0.036; visual mesh filename=package://ur5controller/ur5_description/robotiq_two_finger_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 scale=0.001 0.001 0.001
- link simple_gripper_left_spring_link: geometry collision box size=0.04 0.02 0.065; visual mesh filename=package://ur5controller/ur5_description/robotiq_two_finger_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 scale=0.001 0.001 0.001
- link simple_gripper_right_coupler: geometry collision box size=0.03 0.065 0.02; visual mesh filename=package://ur5controller/ur5_description/robotiq_two_finger_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 scale=0.001 0.001 0.001
- link simple_gripper_right_driver: geometry collision box size=0.02 0.04 0.02; visual mesh filename=package://ur5controller/ur5_description/robotiq_two_finger_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 scale=0.001 0.001 0.001
- link simple_gripper_right_follower: geometry collision box size=0.02 0.015 0.048; visual mesh filename=package://ur5controller/ur5_description/robotiq_two_finger_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 scale=0.001 0.001 0.001
- link simple_gripper_right_pad: geometry collision box size=0.02 0.008 0.036; visual mesh filename=package://ur5controller/ur5_description/robotiq_two_finger_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 scale=0.001 0.001 0.001
- link simple_gripper_right_spring_link: geometry collision box size=0.04 0.02 0.065; visual mesh filename=package://ur5controller/ur5_description/robotiq_two_finger_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 scale=0.001 0.001 0.001
- link upper_arm_link: geometry collision mesh filename=package://ur5controller/ur5_description/arm/meshes/collisio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; visual mesh filename=package://ur5controller/ur5_description/arm/meshes/visual/u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
- link wrist_1_link: geometry collision mesh filename=package://ur5controller/ur5_description/arm/meshes/collisio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; visual mesh filename=package://ur5controller/ur5_description/arm/meshes/visual/w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
- link wrist_2_link: geometry collision mesh filename=package://ur5controller/ur5_description/arm/meshes/collisio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; visual mesh filename=package://ur5controller/ur5_description/arm/meshes/visual/w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
- link wrist_3_link: geometry collision mesh filename=package://ur5controller/ur5_description/arm/meshes/collisio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; visual mesh filename=package://ur5controller/ur5_description/arm/meshes/visual/w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

Commit message: Added ridgeback moving base to the robot model

File: ur5_description/ur5.urdf (robot description, URDF)
Before this commit: robot ur5, 21 links, 20 joints
Links:
- added link arm_stand_link; collision mesh filename=package://ur5controller/ur5_description/ridgeback/arm_stand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; visual mesh filename=package://ur5controller/ur5_description/ridgeback/arm_stand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
- added link axle_link; visual mesh filename=package://ur5controller/ur5_description/ridgeback/axle.stl
- added link base_computer_box_link; collision mesh filename=package://ur5controller/ur5_description/ridgeback/base_comp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; visual mesh filename=package://ur5controller/ur5_description/ridgeback/base_comp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
- added link chassis_link, mass 165.304; collision mesh filename=package://ur5controller/ur5_description/ridgeback/body-coll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; visual mesh filename=package://ur5controller/ur5_description/ridgeback/body.stl
- added link front_cover_link; visual mesh filename=package://ur5controller/ur5_description/ridgeback/end-cover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
- added link front_left_wheel_link, mass 2.3; collision cylinder length=0.079 radius=0.0759; visual mesh filename=package://ur5controller/ur5_description/ridgeback/wheel.stl
- added link front_lights_link; visual mesh filename=package://ur5controller/ur5_description/ridgeback/lights.stl
- added link front_right_wheel_link, mass 2.3; collision cylinder length=0.079 radius=0.0759; visual mesh filename=package://ur5controller/ur5_description/ridgeback/wheel.stl
- added link front_rocker_link, mass 10.267; visual mesh filename=package://ur5controller/ur5_description/ridgeback/rocker.stl
- added link imu_link, mass 0.001
- added link left_side_cover_link; visual mesh filename=package://ur5controller/ur5_description/ridgeback/side-cove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
- added link mid_mount
- added link rear_cover_link; visual mesh filename=package://ur5controller/ur5_description/ridgeback/end-cover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
- added link rear_left_wheel_link, mass 2.3; collision cylinder length=0.079 radius=0.0759; visual mesh filename=package://ur5controller/ur5_description/ridgeback/wheel.stl
- added link rear_lights_link; visual mesh filename=package://ur5controller/ur5_description/ridgeback/lights.stl
- added link rear_right_wheel_link, mass 2.3; collision cylinder length=0.079 radius=0.0759; visual mesh filename=package://ur5controller/ur5_description/ridgeback/wheel.stl
- added link rear_rocker_link, mass 10.267; visual mesh filename=package://ur5controller/ur5_description/ridgeback/rocker.stl
- added link ridgeback_base_link
- added link right_side_cover_link; visual mesh filename=package://ur5controller/ur5_description/ridgeback/side-cove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
- added link top_link; collision mesh filename=package://ur5controller/ur5_description/ridgeback/top.stl; visual mesh filename=package://ur5controller/ur5_description/ridgeback/top.stl
Joints:
- added joint arm_stand_joint: type fixed, parent ridgeback_base_link, child arm_stand_link, origin xyz=-3.703 9 0.28 rpy=0 0 0
- added joint axle_joint: type fixed, parent chassis_link, child axle_link, origin xyz=0 0 0.05 rpy=0 0 0
- added joint base_computer_box_joint: type fixed, parent ridgeback_base_link, child base_computer_box_link, origin xyz=1.35 2.5 -16.72 rpy=0 0 0
- added joint base_link_joint: type fixed, parent ridgeback_base_link, child chassis_link, origin xyz=0 0 0 rpy=0 0 0
- added joint front_cover_link_joint: type fixed, parent chassis_link, child front_cover_link, origin xyz=0 0 0 rpy=0 0 0
- added joint front_left_wheel: type continuous, parent front_rocker_link, child front_left_wheel_link, origin xyz=0 0.2755 0 rpy=0 0 0, axis 0 1 0
- added joint front_lights_link_joint: type fixed, parent chassis_link, child front_lights_link, origin xyz=0 0 0 rpy=0 0 0
- added joint front_right_wheel: type continuous, parent front_rocker_link, child front_right_wheel_link, origin xyz=0 -0.2755 0 rpy=0 0 0, axis 0 1 0
- added joint front_rocker: type revolute, parent axle_link, child front_rocker_link, origin xyz=0.319 0 0 rpy=0 0 0, axis 1 0 0, limit lower=-0.08726 upper=0.08726 effort=0 velocity=0
- added joint imu_joint: type fixed, parent chassis_link, child imu_link, origin xyz=0.2085 -0.2902 0.1681 rpy=0 0 0
- added joint left_side_cover_link_joint: type fixed, parent chassis_link, child left_side_cover_link, origin xyz=0 0 0 rpy=0 0 0
- added joint mid_mount_joint: type fixed, parent ridgeback_base_link, child mid_mount, origin xyz=0 0 0.28 rpy=0 0 0
- added joint rear_cover_link_joint: type fixed, parent chassis_link, child rear_cover_link, origin xyz=0 0 0 rpy=0 0 0
- added joint rear_left_wheel: type continuous, parent rear_rocker_link, child rear_left_wheel_link, origin xyz=0 0.2755 0 rpy=0 0 0, axis 0 1 0
- added joint rear_lights_link_joint: type fixed, parent chassis_link, child rear_lights_link, origin xyz=0 0 0 rpy=0 0 0
- added joint rear_right_wheel: type continuous, parent rear_rocker_link, child rear_right_wheel_link, origin xyz=0 -0.2755 0 rpy=0 0 0, axis 0 1 0
- added joint rear_rocker: type fixed, parent axle_link, child rear_rocker_link, origin xyz=-0.319 0 0 rpy=0 0 0, axis 1 0 0, limit effort=0 velocity=0
- added joint ridgeback_to_arm_joint: type fixed, parent axle_link, child base_link, origin xyz=0.3 0 0.734 rpy=0 0 -1.57
- added joint right_side_cover_link_joint: type fixed, parent chassis_link, child right_side_cover_link, origin xyz=0 0 0 rpy=0 0 0
- added joint top_link_joint: type fixed, parent chassis_link, child top_link, origin xyz=0 0 0 rpy=0 0 0

Commit message: Removed the DOF from the base

File: ur5_description/ur5.urdf (robot description, URDF)
Before this commit: robot ur5, 41 links, 40 joints
Joints:
- joint front_left_wheel: type continuous -> fixed
- joint front_right_wheel: type continuous -> fixed
- joint front_rocker: type revolute -> fixed
- joint rear_left_wheel: type continuous -> fixed
- joint rear_right_wheel: type continuous -> fixed

Commit message: Fixed URDF to place UR5 to correct position; refactoring to ur5controller.cpp

File: ur5_description/ur5.urdf (robot description, URDF)
Before this commit: robot ur5, 41 links, 40 joints
Links:
- link arm_stand_link: geometry collision cylinder length=0.459 radius=0.1; visual cylinder length=0.459 radius=0.1
Joints:
- removed joint ridgeback_to_arm_joint
- added joint arm_stand_to_arm_joint: type fixed, parent arm_stand_link, child base_link, origin xyz=0.0 0.0 0.462 rpy=0 0 -1.57
- joint arm_stand_joint: origin xyz=-3.703 9 0.28 rpy=0 0 0 -> xyz=0.28 0.0 0.0 rpy=0 0 0; parent ridgeback_base_link -> mid_mount

Commit message: Added torque and force sensore (broken)

File: ur5_description/ur5.urdf (robot description, URDF)
Before this commit: robot ur5, 41 links, 40 joints
Links:
- added link arm_to_force_torque_sensor_link; collision box size=0.088 0.088 0.0125; visual box size=0.088 0.088 0.0125
- added link robotiq_force_torque_frame_id
- added link robotiq_fts_robotside, mass 0.65; collision mesh filename=package://ur5controller/ur5_description/robotiq_force_torqu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; visual mesh filename=package://ur5controller/ur5_description/robotiq_force_torqu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
- added link robotiq_fts_toolside
Joints:
- added joint arm_to_force_torque_sensor_joint: type fixed, parent tool0, child arm_to_force_torque_sensor_link, origin xyz=0.0 0.0 0.00625 rpy=0 0 0
- added joint robotiq_fts_fix: type fixed, parent arm_to_force_torque_sensor_link, child robotiq_fts_robotside, origin xyz=0.0 0.0 0.00625 rpy=0 0 0
- added joint robotiq_measurment_joint: type fixed, parent robotiq_fts_robotside, child robotiq_force_torque_frame_id, origin xyz=0 0 0.01625 rpy=0 0 0
- added joint robotiq_toolside_joint: type fixed, parent robotiq_fts_robotside, child robotiq_fts_toolside, origin xyz=0 0 0.0375 rpy=0 0 0
- joint ee_fixed_joint: origin xyz=0.0 0.1623 0.0 rpy=0.0 0.0 1.570796325 -> xyz=0.0 0.0 0.08 rpy=0.0 0.0 1.57075; parent wrist_3_link -> robotiq_fts_toolside

Commit message: Fixed force torque sensor; Now integrated with the ee

File: ur5_description/ur5.urdf (robot description, URDF)
Before this commit: robot ur5, 45 links, 44 joints
Joints:
- joint ee_fixed_joint: origin xyz=0.0 0.0 0.08 rpy=0.0 0.0 1.57075 -> xyz=0.0 0.0 0.08 rpy=1.570796325 -1.570796325 0.0
