Commit message: Minor changes

File: ur5_description/urdf/clearpath_ridgeback__ur5__robotiq_two_finger_gripper.urdf (robot description, URDF)
Before this commit: robot ur5, 41 links, 40 joints
Links:
- link arm_stand_link: geometry collision cylinder length=0.459 radius=0.1; visual cylinder length=0.459 radius=0.1
Joints:
- removed joint ridgeback_to_arm_joint
- added joint arm_stand_to_arm_joint: type fixed, parent arm_stand_link, child base_link, origin xyz=0.0 0.0 0.462 rpy=0 0 -1.57
- joint arm_stand_joint: origin xyz=-3.703 9 0.28 rpy=0 0 0 -> xyz=0.28 0.0 0.0 rpy=0 0 0; parent ridgeback_base_link -> mid_mount
- joint simple_gripper_right_driver_joint: limit lower=0.0 upper=0.872664444444 effort=60 velocity=1.91986177778 -> lower=0.0 upper=0.77 effort=60 velocity=1.91986177778

Commit message: Fixed a minor problem with OpenRAVE warning when opening or closing the gripper.

File: ur5_description/urdf/clearpath_ridgeback__ur5__robotiq_two_finger_gripper.urdf (robot description, URDF)
Before this commit: robot ur5, 41 links, 40 joints
Joints:
- joint simple_gripper_right_driver_joint: limit lower=0.0 upper=0.77 effort=60 velocity=1.91986177778 -> lower=0.0 upper=0.715584844444 effort=60 velocity=1.91986177778

Commit message: Made the computer base box which was too large and causes manipulation problems smaller.

File: ur5_description/urdf/clearpath_ridgeback__ur5__robotiq_two_finger_gripper.urdf (robot description, URDF)
Before this commit: robot ur5, 41 links, 40 joints
Links:
- link base_computer_box_link: geometry collision box size=0.4 0.6 0.6; visual box size=0.4 0.6 0.6

Commit message: Moved the robot cordinate frame from bottom to the top plate surface.
This is for the ridgeback, with two finger gripper and without the force torque sensor.

File: ur5_description/urdf/clearpath_ridgeback__ur5__robotiq_two_finger_gripper.urdf (robot description, URDF)
Before this commit: robot ur5, 41 links, 40 joints
Joints:
- joint arm_stand_joint: origin xyz=0.28 0.0 0.0 rpy=0 0 0 -> xyz=0.28 0.0 -0.28 rpy=0 0 0
- joint base_computer_box_joint: origin xyz=1.35 2.5 -16.72 rpy=0 0 0 -> xyz=1.35 2.5 -17 rpy=0 0 0
- joint base_link_joint: origin xyz=0 0 0 rpy=0 0 0 -> xyz=0 0 -0.28 rpy=0 0 0

Commit message: Minor fix to the model.

File: ur5_description/urdf/clearpath_ridgeback__ur5__robotiq_two_finger_gripper.urdf (robot description, URDF)
Before this commit: robot ur5, 41 links, 40 joints
Joints:
- joint arm_stand_to_arm_joint: origin xyz=0.0 0.0 0.462 rpy=0 0 -1.57 -> xyz=0.0 0.0 0.456 rpy=0 0 -1.57

Commit message: Fixed a rotation error causing ee offsets.

File: ur5_description/urdf/clearpath_ridgeback__ur5__robotiq_two_finger_gripper.urdf (robot description, URDF)
Before this commit: robot ur5, 41 links, 40 joints
Joints:
- joint arm_stand_to_arm_joint: origin xyz=0.0 0.0 0.456 rpy=0 0 -1.57 -> xyz=0.0 0.0 0.456 rpy=0 0 -1.6231562043547265

Commit message: Further rotation to the base of the robot added.

File: ur5_description/urdf/clearpath_ridgeback__ur5__robotiq_two_finger_gripper.urdf (robot description, URDF)
Before this commit: robot ur5, 41 links, 40 joints
Joints:
- joint arm_stand_to_arm_joint: origin xyz=0.0 0.0 0.456 rpy=0 0 -1.6231562043547265 -> xyz=0.0 0.0 0.456 rpy=0 0 -1.64060949685

Commit message: Remove 1 degree from wrist3 joint limits.
When executing trajectories, sometimes the robot was getting into protective stop because was reaching a joint limit.

File: ur5_description/urdf/clearpath_ridgeback__ur5__robotiq_two_finger_gripper.urdf (robot description, URDF)
Before this commit: robot ur5, 41 links, 40 joints
Joints:
- joint wrist_3_joint: limit lower=-6.2831853 upper=6.2831853 effort=28.0 velocity=3.2 -> lower=-6.26573 upper=6.26573 effort=28.0 velocity=3.2

Commit message: Removed 1 degree from all joints.
Due to robot's low-level controller not allowing max or min joint values, we have removed 1 degree from the max and min joint value of each joint.

File: ur5_description/urdf/clearpath_ridgeback__ur5__robotiq_two_finger_gripper.urdf (robot description, URDF)
Before this commit: robot ur5, 41 links, 40 joints
Joints:
- joint elbow_joint: limit lower=-6.2831853 upper=6.2831853 effort=150.0 velocity=3.15 -> lower=-6.26573 upper=6.26573 effort=150.0 velocity=3.15
- joint shoulder_lift_joint: limit lower=-6.2831853 upper=6.2831853 effort=150.0 velocity=3.15 -> lower=-6.26573 upper=6.26573 effort=150.0 velocity=3.15
- joint shoulder_pan_joint: limit lower=-6.2831853 upper=6.2831853 effort=150.0 velocity=3.15 -> lower=-6.26573 upper=6.26573 effort=150.0 velocity=3.15
- joint wrist_1_joint: limit lower=-6.2831853 upper=6.2831853 effort=28.0 velocity=3.2 -> lower=-6.26573 upper=6.26573 effort=28.0 velocity=3.2
- joint wrist_2_joint: limit lower=-6.2831853 upper=6.2831853 effort=28.0 velocity=3.2 -> lower=-6.26573 upper=6.26573 effort=28.0 velocity=3.2

Commit message: Added .stl objects for UR5 stand and computer box.
or_urdf has trouble rendering geometric shapes like boxes and cylinders, as a result the solution to have correct visualisation of the model is to provide a mesh file instead.

File: ur5_description/urdf/clearpath_ridgeback__ur5__robotiq_two_finger_gripper.urdf (robot description, URDF)
Before this commit: robot ur5, 41 links, 40 joints
Links:
- link arm_stand_link: geometry collision mesh filename=package://ur5controller/ur5_description/arm/meshes/visual/a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; visual mesh filename=package://ur5controller/ur5_description/arm/meshes/visual/a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
- link base_computer_box_link: geometry collision mesh filename=package://ur5controller/ur5_description/arm/meshes/visual/c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; visual mesh filename=package://ur5controller/ur5_description/arm/meshes/visual/c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

Commit message: Added inertia information to the gripper.

File: ur5_description/urdf/clearpath_ridgeback__ur5__robotiq_two_finger_gripper.urdf (robot description, URDF)
Before this commit: robot ur5, 41 links, 40 joints
Links:
- link simple_gripper_base: mass None -> 1.267
- link simple_gripper_left_coupler: mass None -> 1.267
- link simple_gripper_left_driver: mass None -> 1.267
- link simple_gripper_left_follower: mass None -> 1.267
- link simple_gripper_left_pad: mass None -> 1.267
- link simple_gripper_left_spring_link: mass None -> 1.267
- link simple_gripper_right_coupler: mass None -> 1.267
- link simple_gripper_right_driver: mass None -> 1.267
- link simple_gripper_right_follower: mass None -> 1.267
- link simple_gripper_right_pad: mass None -> 1.267
- link simple_gripper_right_spring_link: mass None -> 1.267
