Commit message: Fixed an error to collision rotation of the force sensor and added collision safety to the plug of the force sensor.

File: ur5_description/urdf/clearpath_ridgeback__ur5__robotiq_two_finger_gripper__robotiq_fts150.urdf (robot description, URDF)
Before this commit: robot ur5, 45 links, 44 joints
Links:
- added link force_sensor_cable_port_placeholder_link; collision box size=0.07 0.05 0.032; visual box size=0.07 0.05 0.032
Joints:
- added joint force_sensor_cable_port_placeholder_joint: type fixed, parent force_sensor_cable_port_placeholder_link, child robotiq_force_torque_frame_id, origin xyz=0.28 0.0 0.0 rpy=0 0 0
- joint robotiq_measurment_joint: child robotiq_force_torque_frame_id -> force_sensor_cable_port_placeholder_link

Commit message: Added support for open and close gripper to the robot instance.

File: ur5_description/urdf/clearpath_ridgeback__ur5__robotiq_two_finger_gripper__robotiq_fts150.urdf (robot description, URDF)
Before this commit: robot ur5, 46 links, 45 joints
Joints:
- joint simple_gripper_right_driver_joint: limit lower=0.0 upper=0.872664444444 effort=60 velocity=1.91986177778 -> lower=0.0 upper=0.77 effort=60 velocity=1.91986177778

Commit message: Updated the model with FTS150 to be compatible with the others.

File: ur5_description/urdf/clearpath_ridgeback__ur5__robotiq_two_finger_gripper__robotiq_fts150.urdf (robot description, URDF)
Before this commit: robot ur5, 46 links, 45 joints
Links:
- link arm_stand_link: geometry collision mesh filename=package://ur5controller/ur5_description/arm/meshes/visual/a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; visual mesh filename=package://ur5controller/ur5_description/arm/meshes/visual/a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
- link base_computer_box_link: geometry collision mesh filename=package://ur5controller/ur5_description/arm/meshes/visual/c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; visual mesh filename=package://ur5controller/ur5_description/arm/meshes/visual/c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
- link simple_gripper_base: mass None -> 1.267
- link simple_gripper_left_coupler: mass None -> 1.267
- link simple_gripper_left_driver: mass None -> 1.267
- link simple_gripper_left_follower: mass None -> 1.267
- link simple_gripper_left_pad: mass None -> 1.267
- link simple_gripper_left_spring_link: mass None -> 1.267
- link simple_gripper_right_coupler: mass None -> 1.267
- link simple_gripper_right_driver: mass None -> 1.267
- link simple_gripper_right_follower: mass None -> 1.267
- link simple_gripper_right_pad: mass None -> 1.267
- link simple_gripper_right_spring_link: mass None -> 1.267
Joints:
- joint arm_stand_joint: origin xyz=0.28 0.0 0.0 rpy=0 0 0 -> xyz=0.28 0.0 -0.28 rpy=0 0 0
- joint arm_stand_to_arm_joint: origin xyz=0.0 0.0 0.462 rpy=0 0 -1.57 -> xyz=0.0 0.0 0.456 rpy=0 0 -1.64060949685
- joint base_computer_box_joint: origin xyz=1.35 2.5 -16.72 rpy=0 0 0 -> xyz=1.35 2.5 -17 rpy=0 0 0
- joint base_link_joint: origin xyz=0 0 0 rpy=0 0 0 -> xyz=0 0 -0.28 rpy=0 0 0
- joint elbow_joint: limit lower=-6.2831853 upper=6.2831853 effort=150.0 velocity=3.15 -> lower=-6.26573 upper=6.26573 effort=150.0 velocity=3.15
- joint shoulder_lift_joint: limit lower=-6.2831853 upper=6.2831853 effort=150.0 velocity=3.15 -> lower=-6.26573 upper=6.26573 effort=150.0 velocity=3.15
- joint shoulder_pan_joint: limit lower=-6.2831853 upper=6.2831853 effort=150.0 velocity=3.15 -> lower=-6.26573 upper=6.26573 effort=150.0 velocity=3.15
- joint simple_gripper_right_driver_joint: limit lower=0.0 upper=0.77 effort=60 velocity=1.91986177778 -> lower=0.0 upper=0.715584844444 effort=60 velocity=1.91986177778
- joint wrist_1_joint: limit lower=-6.2831853 upper=6.2831853 effort=28.0 velocity=3.2 -> lower=-6.26573 upper=6.26573 effort=28.0 velocity=3.2
- joint wrist_2_joint: limit lower=-6.2831853 upper=6.2831853 effort=28.0 velocity=3.2 -> lower=-6.26573 upper=6.26573 effort=28.0 velocity=3.2
- joint wrist_3_joint: limit lower=-6.2831853 upper=6.2831853 effort=28.0 velocity=3.2 -> lower=-6.26573 upper=6.26573 effort=28.0 velocity=3.2
